File: PCB Design/Sequencer/Sequencer.kicad_sch (KiCad schematic)
At the start: 180 parts, among them SW1 SW_MEC_5G, SW10 SW_MEC_5G, SW11 SW_MEC_5G, SW12 SW_MEC_5G, SW13 SW_MEC_5G, SW14 SW_MEC_5G, SW15 SW_MEC_5G, SW16 SW_MEC_5G, SW2 SW_MEC_5G, SW3 SW_MEC_5G, SW4 SW_MEC_5G, SW5 SW_MEC_5G, SW6 SW_MEC_5G, SW7 SW_MEC_5G, SW8 SW_MEC_5G, SW9 SW_MEC_5G, U27 DM74LS54N, U28 DM74LS54N, U29 DM74LS54N, U30 DM74LS54N

Commit message: Sequencer update
Parts:
- added BEATS_3_1, BEATS_3_2, BEATS_3_3, BEATS_3_4: DM74LS54N, symbol DM74LS54N:DM74LS54N
- added COMBINE_3: ~, symbol MC14012B:MC14012B
- added D_3_1_1, D_3_1_2, D_3_2_1, D_3_2_2, D_3_3_1, D_3_3_2, D_3_4_1, D_3_4_2, D_3_5_1, D_3_5_2, D_3_6_1, D_3_6_2, D_3_7_1, D_3_7_2, D_3_8_1, D_3_8_2: LED, Diode_THT:D_5W_P5.08mm_Vertical_AnodeUp, symbol Device:LED
- added INVERT: ~, symbol DM74LS04N:DM74LS04N
- added JK_3_1, JK_3_2, JK_3_3, JK_3_4, JK_3_5, JK_3_6, JK_3_7, JK_3_8: SN74107N, SN74107N:DIP254P762X508-14, symbol SN74107N:SN74107N
- added OUT_PINS: OUT_PINS, symbol Connector:Conn_01x05_Pin
- added R1: 1M, Resistor_THT:R_Axial_DIN0309_L9.0mm_D3.2mm_P12.70mm_Horizontal, symbol Device:R
- added R2: 100K, Resistor_THT:R_Axial_DIN0309_L9.0mm_D3.2mm_P12.70mm_Horizontal, symbol Device:R
- added R_3_1_1, R_3_1_2, R_3_2_1, R_3_2_2, R_3_3_1, R_3_3_2, R_3_4_1, R_3_4_2, R_3_5_1, R_3_5_2, R_3_6_1, R_3_6_2, R_3_7_1, R_3_7_2, R_3_8_1, R_3_8_2: R, Resistor_THT:R_Axial_DIN0309_L9.0mm_D3.2mm_P12.70mm_Horizontal, symbol Device:R
- renumbered U27 to BEATS_2_1, U28 to BEATS_2_2, U29 to BEATS_2_3, U30 to BEATS_2_4, U31 to COMBINE_2
Connections:
- net +5V: now also BEATS_3_1.14 (VCC), BEATS_3_1.5 (E), BEATS_3_1.9 (F), BEATS_3_2.14 (VCC), BEATS_3_2.5 (E), BEATS_3_2.9 (F), BEATS_3_3.14 (VCC), BEATS_3_3.5 (E), BEATS_3_3.9 (F), BEATS_3_4.14 (VCC), BEATS_3_4.5 (E), BEATS_3_4.9 (F), COMBINE_3.11 (IN_3_B), COMBINE_3.12 (IN_4_B), COMBINE_3.14 (VDD), INVERT.14 (VCC), JK_3_1.10 (2~CLR), JK_3_1.13 (1~CLR), JK_3_1.14 (VCC), JK_3_2.10 (2~CLR), JK_3_2.13 (1~CLR), JK_3_2.14 (VCC), JK_3_3.10 (2~CLR), JK_3_3.13 (1~CLR), JK_3_3.14 (VCC), JK_3_4.10 (2~CLR), JK_3_4.13 (1~CLR), JK_3_4.14 (VCC), JK_3_5.10 (2~CLR), JK_3_5.13 (1~CLR), JK_3_5.14 (VCC), JK_3_6.10 (2~CLR), JK_3_6.13 (1~CLR), JK_3_6.14 (VCC), JK_3_7.10 (2~CLR), JK_3_7.13 (1~CLR), JK_3_7.14 (VCC), JK_3_8.10 (2~CLR), JK_3_8.13 (1~CLR), JK_3_8.14 (VCC), R1.2
- net GND: now also BEATS_3_1.7 (GND), BEATS_3_2.7 (GND), BEATS_3_3.7 (GND), BEATS_3_4.7 (GND), COMBINE_3.7 (VSS), INVERT.7 (GND), JK_3_1.7 (GND), JK_3_2.7 (GND), JK_3_3.7 (GND), JK_3_4.7 (GND), JK_3_5.7 (GND), JK_3_6.7 (GND), JK_3_7.7 (GND), JK_3_8.7 (GND), OUT_PINS.1 (Pin_1), R2.2, R_3_1_1.1, R_3_1_2.1, R_3_2_1.1, R_3_2_2.1, R_3_3_1.1, R_3_3_2.1, R_3_4_1.1, R_3_4_2.1, R_3_5_1.1, R_3_5_2.1, R_3_6_1.1, R_3_6_2.1, R_3_7_1.1, R_3_7_2.1, R_3_8_1.1, R_3_8_2.1
- net at C7.1, JK_1_3.12 (1CLK), JK_2_3.12 (1CLK)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: now also JK_3_3.12 (1CLK)
- net at BEATS_1_3.12 (I), BEATS_2_3.12 (I), D27.2 (A)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: now also BEATS_3_3.12 (I)
- net at C17.1, JK_1_8.12 (1CLK), JK_2_8.12 (1CLK)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: now also JK_3_8.12 (1CLK)
- net at C8.1, JK_1_3.9 (2CLK), JK_2_3.9 (2CLK)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: now also JK_3_3.9 (2CLK)
- net at BEATS_1_4.12 (I), BEATS_2_4.12 (I), D31.2 (A)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: now also BEATS_3_4.12 (I)
- net at BEATS_1_1.12 (I), BEATS_2_1.12 (I), D19.2 (A)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: now also BEATS_3_1.12 (I)
- net at C9.1, JK_1_4.12 (1CLK), JK_2_4.12 (1CLK)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: now also JK_3_4.12 (1CLK)
- net at C11.1, JK_1_5.12 (1CLK), JK_2_5.12 (1CLK)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: now also JK_3_5.12 (1CLK)
- net at C3.1, JK_1_1.12 (1CLK), JK_2_1.12 (1CLK)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: now also JK_3_1.12 (1CLK)
- net at C4.1, JK_1_1.9 (2CLK), JK_2_1.9 (2CLK)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: now also JK_3_1.9 (2CLK)
- net at C6.1, JK_1_2.9 (2CLK), JK_2_2.9 (2CLK)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: now also JK_3_2.9 (2CLK)
- net at C16.1, JK_1_7.9 (2CLK), JK_2_7.9 (2CLK)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: now also JK_3_7.9 (2CLK)
- net at C10.1, JK_1_4.9 (2CLK), JK_2_4.9 (2CLK)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: now also JK_3_4.9 (2CLK)
- net at C14.1, JK_1_6.9 (2CLK), JK_2_6.9 (2CLK)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: now also JK_3_6.9 (2CLK)
- net at C13.1, JK_1_6.12 (1CLK), JK_2_6.12 (1CLK)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: now also JK_3_6.12 (1CLK)
- net at BEATS_1_3.10 (G), BEATS_2_3.10 (G), D28.2 (A)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: now also BEATS_3_3.10 (G)
- net at BEATS_1_3.2 (B), BEATS_2_3.2 (B), D25.2 (A)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: now also BEATS_3_3.2 (B)
- net at BEATS_1_3.4 (D), BEATS_2_3.4 (D), D26.2 (A)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: now also BEATS_3_3.4 (D)
- net at C5.1, JK_1_2.12 (1CLK), JK_2_2.12 (1CLK)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: now also JK_3_2.12 (1CLK)
- net at BEATS_1_2.2 (B), BEATS_2_2.2 (B), D21.2 (A)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: now also BEATS_3_2.2 (B)
- net at BEATS_1_2.4 (D), BEATS_2_2.4 (D), D22.2 (A)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: now also BEATS_3_2.4 (D)
- net at BEATS_1_2.12 (I), BEATS_2_2.12 (I), D23.2 (A)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: now also BEATS_3_2.12 (I)
- net at BEATS_1_2.10 (G), BEATS_2_2.10 (G), D24.2 (A)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: now also BEATS_3_2.10 (G)
- net at BEATS_1_1.2 (B), BEATS_2_1.2 (B), D17.2 (A)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: now also BEATS_3_1.2 (B)
- net at BEATS_1_1.4 (D), BEATS_2_1.4 (D), D18.2 (A)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: now also BEATS_3_1.4 (D)
- net at BEATS_1_1.10 (G), BEATS_2_1.10 (G), D20.2 (A)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: now also BEATS_3_1.10 (G)
- net at COMBINE_1.9 (IN_1_B), COMBINE_2.9 (IN_1_B), TEMPO.3 (Q)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: now also COMBINE_3.9 (IN_1_B)
- net at BEATS_1_4.4 (D), BEATS_2_4.4 (D), D30.2 (A)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: now also BEATS_3_4.4 (D)
- net at C12.1, JK_1_5.9 (2CLK), JK_2_5.9 (2CLK)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: now also JK_3_5.9 (2CLK)
- net at C18.1, JK_1_8.9 (2CLK), JK_2_8.9 (2CLK)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: now also JK_3_8.9 (2CLK)
- net at C15.1, JK_1_7.12 (1CLK), JK_2_7.12 (1CLK)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: now also JK_3_7.12 (1CLK)
- net at BEATS_1_4.10 (G), BEATS_2_4.10 (G), D32.2 (A)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: now also BEATS_3_4.10 (G)
- net at BEATS_1_4.2 (B), BEATS_2_4.2 (B), D29.2 (A)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: now also BEATS_3_4.2 (B)
- net at COMBINE_1.13 (OUT_B): now also INVERT.1 (A1)
- net at COMBINE_2.13 (OUT_B): now also INVERT.3 (A2)
- new net: D_3_8_1.1 (K), R_3_8_1.2
- new net: D_3_1_2.1 (K), R_3_1_2.2
- new net: BEATS_3_4.1 (A), D_3_7_1.2 (A), JK_3_7.3 (1Q)
- new net: BEATS_3_4.11 (H), D_3_8_2.2 (A), JK_3_8.5 (2Q)
- new net: BEATS_3_4.13 (J), D_3_8_1.2 (A), JK_3_8.3 (1Q)
- new net: BEATS_3_4.3 (C), D_3_7_2.2 (A), JK_3_7.5 (2Q)
- new net: BEATS_3_4.6 (Y), COMBINE_3.5 (IN_4_A)
- new net: BEATS_3_1.1 (A), D_3_1_1.2 (A), JK_3_1.3 (1Q)
- new net: BEATS_3_1.11 (H), D_3_2_2.2 (A), JK_3_2.5 (2Q)
- new net: BEATS_3_1.13 (J), D_3_2_1.2 (A), JK_3_2.3 (1Q)
- new net: BEATS_3_1.3 (C), D_3_1_2.2 (A), JK_3_1.5 (2Q)
- new net: BEATS_3_1.6 (Y), COMBINE_3.2 (IN_1_A)
- new net: D_3_3_1.1 (K), R_3_3_1.2
- new net: BEATS_3_2.1 (A), D_3_3_1.2 (A), JK_3_3.3 (1Q)
- new net: BEATS_3_2.11 (H), D_3_4_2.2 (A), JK_3_4.5 (2Q)
- new net: BEATS_3_2.13 (J), D_3_4_1.2 (A), JK_3_4.3 (1Q)
- new net: BEATS_3_2.3 (C), D_3_3_2.2 (A), JK_3_3.5 (2Q)
- new net: BEATS_3_2.6 (Y), COMBINE_3.3 (IN_2_A)
- new net: D_3_1_1.1 (K), R_3_1_1.2
- new net: JK_3_1.1 (1J), JK_3_1.11 (2K), JK_3_1.4 (1K), JK_3_1.8 (2J), JK_3_2.1 (1J), JK_3_2.11 (2K), JK_3_2.4 (1K), JK_3_2.8 (2J), JK_3_3.1 (1J), JK_3_3.11 (2K), JK_3_3.4 (1K), JK_3_3.8 (2J), JK_3_4.1 (1J), JK_3_4.11 (2K), JK_3_4.4 (1K), JK_3_4.8 (2J), JK_3_5.1 (1J), JK_3_5.11 (2K), JK_3_5.4 (1K), JK_3_5.8 (2J), JK_3_6.1 (1J), JK_3_6.11 (2K), JK_3_6.4 (1K), JK_3_6.8 (2J), JK_3_7.1 (1J), JK_3_7.11 (2K), JK_3_7.4 (1K), JK_3_7.8 (2J), JK_3_8.1 (1J), JK_3_8.11 (2K), JK_3_8.4 (1K), JK_3_8.8 (2J)
- new net: OUT_PINS.2 (Pin_2), R1.1, R2.1
- new net: D_3_4_1.1 (K), R_3_4_1.2
- new net: D_3_4_2.1 (K), R_3_4_2.2
- new net: BEATS_3_3.1 (A), D_3_5_1.2 (A), JK_3_5.3 (1Q)
- new net: BEATS_3_3.3 (C), D_3_5_2.2 (A), JK_3_5.5 (2Q)
- new net: D_3_8_2.1 (K), R_3_8_2.2
- new net: D_3_6_1.1 (K), R_3_6_1.2
- new net: D_3_2_1.1 (K), R_3_2_1.2
- new net: BEATS_3_3.13 (J), D_3_6_1.2 (A), JK_3_6.3 (1Q)
- new net: D_3_3_2.1 (K), R_3_3_2.2
- new net: D_3_5_2.1 (K), R_3_5_2.2
- new net: INVERT.2 (Y1), OUT_PINS.3 (Pin_3)
- new net: INVERT.4 (Y2), OUT_PINS.4 (Pin_4)
- new net: INVERT.6 (Y3), OUT_PINS.5 (Pin_5)
- new net: D_3_5_1.1 (K), R_3_5_1.2
- new net: D_3_7_2.1 (K), R_3_7_2.2
- new net: BEATS_3_3.11 (H), D_3_6_2.2 (A), JK_3_6.5 (2Q)
- new net: D_3_6_2.1 (K), R_3_6_2.2
- new net: D_3_2_2.1 (K), R_3_2_2.2
- new net: COMBINE_3.13 (OUT_B), INVERT.5 (A3)
- new net: BEATS_3_3.6 (Y), COMBINE_3.4 (IN_3_A)
- new net: D_3_7_1.1 (K), R_3_7_1.2
- new net: COMBINE_3.1 (OUT_A), COMBINE_3.10 (IN_2_B)
- no-connect marks 42 -> 58

Commit message: Sequencer update
Parts:
- removed D17, D18, D19, D20, D21, D22, D23, D24, D25, D26, D27, D28, D29, D30, D31, D32: LED, Diode_THT:D_5W_P5.08mm_Vertical_AnodeUp, symbol Device:LED
- removed R19, R20, R21, R22, R23, R24, R25, R26, R27, R28, R29, R30, R31, R32, R33, R34: R, Resistor_THT:R_Axial_DIN0309_L9.0mm_D3.2mm_P12.70mm_Horizontal, symbol Device:R
- BEATS_1_1, BEATS_1_2, BEATS_1_3, BEATS_1_4, BEATS_2_1, BEATS_2_2, BEATS_2_3, BEATS_2_4, BEATS_3_1, BEATS_3_2, BEATS_3_3, BEATS_3_4: footprint (none) -> DM74LS54N:DM74LS54N
- COMBINE_1, COMBINE_2, COMBINE_3: footprint (none) -> MC14012B:MC14012B
- INVERT: footprint (none) -> DM74LS04N:DM74LS04N
- JK_2_1, JK_2_2, JK_2_3, JK_2_4, JK_2_5, JK_2_6, JK_2_7, JK_2_8, JK_3_1, JK_3_2, JK_3_3, JK_3_4, JK_3_5, JK_3_6, JK_3_7, JK_3_8: footprint SN74107N:DIP254P762X508-14 -> SN74107N:SN74107N
- ONE_SHOT: renamed from U16; footprint (none) -> SN74LS95BN:SN74LS95BN
- R_Tempo: renamed from RV1; value R_Pot -> 2M
- SHIFT_1: renamed from U15; footprint (none) -> DM74164N:DM74164N
- SHIFT_2: renamed from U14; footprint (none) -> DM74164N:DM74164N
- XOR: renamed from U17; footprint (none) -> CD4070BE:CD4070BE
- renumbered TEMPO to 555_TIMER, R17 to R1, R18 to R2, R1 to R3, R2 to R4
Connections:
- net +5V: no longer ONE_SHOT.14 (VCC)
- net GND: no longer ONE_SHOT.1 (SER), ONE_SHOT.6 (MODE), ONE_SHOT.7 (GND)
- net at 555_TIMER.3 (Q), COMBINE_1.9 (IN_1_B), COMBINE_2.9 (IN_1_B)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: no longer ONE_SHOT.9 (CLK1)
- net at ONE_SHOT.12 (Q_B): no longer XOR.8 (E)
- net at ONE_SHOT.13 (Q_A): no longer XOR.9 (F)
- net at COMBINE_1.13 (OUT_B): now also INVERT.3 (A2); no longer INVERT.1 (A1)
- net at COMBINE_2.13 (OUT_B): now also INVERT.1 (A1); no longer INVERT.3 (A2)
- no-connect marks 58 -> 64
Other:
- note added: "OUT_PINS POTENTIOMETER BUTTONS POWER GANGED SWITCH"
- moved on the sheet: INVERT

Commit message: Sequencer complete schematic w/o values
Parts:
- removed R37, R38, R39, R40, R41, R42, R43, R44, R45, R46, R47, R48, R49, R50: R, symbol Device:R
- added 5V_POWER: Barrel_Jack_Switch, symbol Connector:Barrel_Jack_Switch
- added DISABLER: GANGED_SW_SP3T, symbol Switch:SW_SP3T
- added R10, R11, R12, R13, R14, R15, R16, R17, R18, R19, R20, R21, R22, R23, R24, R25, R26, R27, R28, R29, R30, R31, R32, R33, R34, R5, R6, R7, R8, R9: R, symbol Device:R
- OUT_PINS: footprint (none) -> Connector_PinHeader_1.00mm:PinHeader_1x05_P1.00mm_Vertical
- R_Tempo: footprint (none) -> Potentiometer_THT:Potentiometer_Omeg_PC16BU_Vertical
Connections:
- net +5V: now also 5V_POWER.1, R11.1, R22.1, R23.1, R24.1, R25.1, R26.1, R27.1, R28.1, R29.1, R30.1, R31.1, R32.1, R33.1, R34.1
- net GND: now also SW1.3 (B), SW1.4 (B), SW10.3 (B), SW10.4 (B), SW11.3 (B), SW11.4 (B), SW12.3 (B), SW12.4 (B), SW13.3 (B), SW13.4 (B), SW14.3 (B), SW14.4 (B), SW15.3 (B), SW15.4 (B), SW16.3 (B), SW16.4 (B), SW2.3 (B), SW2.4 (B), SW3.3 (B), SW3.4 (B), SW4.3 (B), SW4.4 (B), SW5.3 (B), SW5.4 (B), SW6.3 (B), SW6.4 (B), SW7.3 (B), SW7.4 (B), SW8.3 (B), SW8.4 (B), SW9.3 (B), SW9.4 (B), 5V_POWER.2, 5V_POWER.3, DISABLER.7, R10.1, R12.1, R13.1, R14.1, R15.1, R16.1, R17.1, R18.1, R19.1, R20.1, R21.1, R5.1, R6.1, R7.1, R8.1, R9.1; no longer SW1.1 (A), SW1.2 (A), SW10.1 (A), SW10.2 (A), SW11.1 (A), SW11.2 (A), SW12.1 (A), SW12.2 (A), SW13.1 (A), SW13.2 (A), SW14.1 (A), SW14.2 (A), SW15.1 (A), SW15.2 (A), SW16.1 (A), SW16.2 (A), SW2.1 (A), SW2.2 (A), SW3.1 (A), SW3.2 (A), SW4.1 (A), SW4.2 (A), SW5.1 (A), SW5.2 (A), SW6.1 (A), SW6.2 (A), SW7.1 (A), SW7.2 (A), SW8.1 (A), SW8.2 (A), SW9.1 (A), SW9.2 (A)
- net at C7.1, JK_1_3.12 (1CLK), JK_2_3.12 (1CLK)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: now also SW5.1 (A), SW5.2 (A), R24.2; no longer SW5.3 (B), SW5.4 (B)
- net at C17.1, JK_1_8.12 (1CLK), JK_2_8.12 (1CLK)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: now also SW15.1 (A), SW15.2 (A), R34.2; no longer SW15.3 (B), SW15.4 (B)
- net at C8.1, JK_1_3.9 (2CLK), JK_2_3.9 (2CLK)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: now also SW6.1 (A), SW6.2 (A), R25.2; no longer SW6.3 (B), SW6.4 (B)
- net at C9.1, JK_1_4.12 (1CLK), JK_2_4.12 (1CLK)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: now also SW7.1 (A), SW7.2 (A), R26.2; no longer SW7.3 (B), SW7.4 (B)
- net at C11.1, JK_1_5.12 (1CLK), JK_2_5.12 (1CLK)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: now also SW9.1 (A), SW9.2 (A), R28.2; no longer SW9.3 (B), SW9.4 (B)
- net at JK_1_1.1 (1J), JK_1_1.11 (2K), JK_1_1.4 (1K)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: now also DISABLER.4, DISABLER.5
- net at C3.1, JK_1_1.12 (1CLK), JK_2_1.12 (1CLK)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: now also SW1.1 (A), SW1.2 (A); no longer SW1.3 (B), SW1.4 (B)
- net at C4.1, JK_1_1.9 (2CLK), JK_2_1.9 (2CLK)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: now also SW2.1 (A), SW2.2 (A), R11.2; no longer R36.2, SW2.3 (B), SW2.4 (B)
- net at C6.1, JK_1_2.9 (2CLK), JK_2_2.9 (2CLK)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: now also SW4.1 (A), SW4.2 (A), R23.2; no longer SW4.3 (B), SW4.4 (B)
- net at BEATS_1_4.10 (G), BEATS_2_4.10 (G), BEATS_3_4.10 (G)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: now also SW16.5 (VCC)
- net at BEATS_1_4.12 (I), BEATS_2_4.12 (I), BEATS_3_4.12 (I)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: now also SW15.5 (VCC)
- net at BEATS_1_4.2 (B), BEATS_2_4.2 (B), BEATS_3_4.2 (B)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: now also SW13.5 (VCC)
- net at BEATS_1_4.4 (D), BEATS_2_4.4 (D), BEATS_3_4.4 (D)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: now also SW14.5 (VCC)
- net at C16.1, JK_1_7.9 (2CLK), JK_2_7.9 (2CLK)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: now also SW14.1 (A), SW14.2 (A), R33.2; no longer SW14.3 (B), SW14.4 (B)
- net at BEATS_1_1.10 (G), BEATS_2_1.10 (G), BEATS_3_1.10 (G)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: now also SW4.5 (VCC)
- net at BEATS_1_1.12 (I), BEATS_2_1.12 (I), BEATS_3_1.12 (I)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: now also SW3.5 (VCC)
- net at BEATS_1_1.2 (B), BEATS_2_1.2 (B), BEATS_3_1.2 (B)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: now also SW1.5 (VCC)
- net at BEATS_1_1.4 (D), BEATS_2_1.4 (D), BEATS_3_1.4 (D)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: now also SW2.5 (VCC)
- net at JK_2_1.1 (1J), JK_2_1.11 (2K), JK_2_1.4 (1K)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: now also DISABLER.1, DISABLER.6
- net at C10.1, JK_1_4.9 (2CLK), JK_2_4.9 (2CLK)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: now also SW8.1 (A), SW8.2 (A), R27.2; no longer SW8.3 (B), SW8.4 (B)
- net at C14.1, JK_1_6.9 (2CLK), JK_2_6.9 (2CLK)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: now also SW12.1 (A), SW12.2 (A), R31.2; no longer SW12.3 (B), SW12.4 (B)
- net at BEATS_1_2.10 (G), BEATS_2_2.10 (G), BEATS_3_2.10 (G)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: now also SW8.5 (VCC)
- net at BEATS_1_2.12 (I), BEATS_2_2.12 (I), BEATS_3_2.12 (I)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: now also SW7.5 (VCC)
- net at BEATS_1_2.2 (B), BEATS_2_2.2 (B), BEATS_3_2.2 (B)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: now also SW5.5 (VCC)
- net at BEATS_1_2.4 (D), BEATS_2_2.4 (D), BEATS_3_2.4 (D)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: now also SW6.5 (VCC)
- net at C13.1, JK_1_6.12 (1CLK), JK_2_6.12 (1CLK)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: now also SW11.1 (A), SW11.2 (A), R30.2; no longer SW11.3 (B), SW11.4 (B)
- net at BEATS_1_3.10 (G), BEATS_2_3.10 (G), BEATS_3_3.10 (G)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: now also SW12.5 (VCC)
- net at BEATS_1_3.12 (I), BEATS_2_3.12 (I), BEATS_3_3.12 (I)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: now also SW11.5 (VCC)
- net at BEATS_1_3.2 (B), BEATS_2_3.2 (B), BEATS_3_3.2 (B)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: now also SW9.5 (VCC)
- net at BEATS_1_3.4 (D), BEATS_2_3.4 (D), BEATS_3_3.4 (D)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: now also SW10.5 (VCC)
- net at JK_3_1.1 (1J), JK_3_1.11 (2K), JK_3_1.4 (1K)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: now also DISABLER.2, DISABLER.3
- net at C15.1, JK_1_7.12 (1CLK), JK_2_7.12 (1CLK)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: now also SW13.1 (A), SW13.2 (A), R32.2; no longer SW13.3 (B), SW13.4 (B)
- net at C5.1, JK_1_2.12 (1CLK), JK_2_2.12 (1CLK)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: now also SW3.1 (A), SW3.2 (A), R22.2; no longer SW3.3 (B), SW3.4 (B)
- net at C12.1, JK_1_5.9 (2CLK), JK_2_5.9 (2CLK)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: now also SW10.1 (A), SW10.2 (A), R29.2; no longer SW10.3 (B), SW10.4 (B)
- net at C18.1, JK_1_8.9 (2CLK), JK_2_8.9 (2CLK)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: now also R36.2, SW16.1 (A), SW16.2 (A); no longer SW16.3 (B), SW16.4 (B)
- net at COMBINE_1.13 (OUT_B): now also INVERT.1 (A1); no longer INVERT.3 (A2)
- net at COMBINE_2.13 (OUT_B): now also INVERT.3 (A2); no longer INVERT.1 (A1)
- new net: R18.2, SW13.6 (B)
- new net: R13.2, SW8.6 (B)
- new net: R16.2, SW11.6 (B)
- new net: R6.2, SW1.6 (B)
- new net: R8.2, SW4.6 (B)
- new net: R14.2, SW9.6 (B)
- new net: R9.2, SW5.6 (B)
- new net: R19.2, SW14.6 (B)
- new net: R5.2, SW2.6 (B)
- new net: R21.2, SW16.6 (B)
- new net: R10.2, SW6.6 (B)
- new net: R15.2, SW10.6 (B)
- new net: R7.2, SW3.6 (B)
- new net: R20.2, SW15.6 (B)
- new net: R17.2, SW12.6 (B)
- new net: R12.2, SW7.6 (B)
Other:
- note added: "PCB: POT? POWER BUTTONS GANGED SWITCH"
- note removed: "OUT_PINS POTENTIOMETER BUTTONS POWER GANGED SWITCH"
- moved on the sheet: 555_TIMER, BEATS_1_1, BEATS_1_2, BEATS_1_3, BEATS_1_4, BEATS_2_1, BEATS_2_2, BEATS_2_3, BEATS_2_4, BEATS_3_1, BEATS_3_2, BEATS_3_3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

Commit message: Initial sequencer PCB
Parts:
- renumbered 555_TIMER to 555_TIMER1, ONE_SHOT to ONE_SHOT1, R_Tempo to R_Tempo1, C12 to SW10_C, R29 to SW10_R1, R15 to SW10_R2, C13 to SW11_C, R30 to SW11_R1, R16 to SW11_R2, C14 to SW12_C, R31 to SW12_R1, R17 to SW12_R2, C15 to SW13_C, R32 to SW13_R1, R18 to SW13_R2, C16 to SW14_C, R33 to SW14_R1, R19 to SW14_R2, C17 to SW15_C, R34 to SW15_R1, R20 to SW15_R2, C18 to SW16_C, R36 to SW16_R1, R21 to SW16_R2, C3 to SW1_C, R35 to SW1_R1, R6 to SW1_R2, C4 to SW2_C, R11 to SW2_R1, R5 to SW2_R2, C5 to SW3_C, R22 to SW3_R1, R7 to SW3_R2, C6 to SW4_C, R23 to SW4_R1, R8 to SW4_R2, C7 to SW5_C, R24 to SW5_R1, R9 to SW5_R2, C8 to SW6_C, R25 to SW6_R1, R10 to SW6_R2, C9 to SW7_C, R26 to SW7_R1, R12 to SW7_R2, C10 to SW8_C, R27 to SW8_R1, R13 to SW8_R2, C11 to SW9_C, R28 to SW9_R1, R14 to SW9_R2, XOR to XOR1
Connections:
- net +5V: now also ONE_SHOT1.14 (VCC), SW10_R1.2, SW12_R1.2, SW14_R1.2, SW16_R1.2, SW2_R1.2, SW4_R1.2, SW6_R1.2, SW8_R1.2; no longer SW10_R1.1, SW12_R1.1, SW14_R1.1, SW16_R1.1, SW2_R1.1, SW4_R1.1, SW6_R1.1, SW8_R1.1
- net GND: now also ONE_SHOT1.1 (SER), ONE_SHOT1.6 (MODE), ONE_SHOT1.7 (GND)
- net at JK_1_4.9 (2CLK), JK_2_4.9 (2CLK), JK_3_4.9 (2CLK)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: now also SW8_R1.1; no longer SW8_R1.2
- net at JK_1_2.9 (2CLK), JK_2_2.9 (2CLK), JK_3_2.9 (2CLK)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: now also SW4_R1.1; no longer SW4_R1.2
- net at JK_1_1.9 (2CLK), JK_2_1.9 (2CLK), JK_3_1.9 (2CLK)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: now also SW2_R1.1; no longer SW2_R1.2
- net at JK_1_8.9 (2CLK), JK_2_8.9 (2CLK), JK_3_8.9 (2CLK)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: now also SW16_R1.1; no longer SW16_R1.2
- net at JK_1_7.9 (2CLK), JK_2_7.9 (2CLK), JK_3_7.9 (2CLK)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: now also SW14_R1.1; no longer SW14_R1.2
- net at JK_1_5.9 (2CLK), JK_2_5.9 (2CLK), JK_3_5.9 (2CLK)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: now also SW10_R1.1; no longer SW10_R1.2
- net at 555_TIMER1.3 (Q), COMBINE_1.9 (IN_1_B), COMBINE_2.9 (IN_1_B)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: now also ONE_SHOT1.9 (CLK1)
- net at JK_1_3.9 (2CLK), JK_2_3.9 (2CLK), JK_3_3.9 (2CLK)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: now also SW6_R1.1; no longer SW6_R1.2
- net at JK_1_6.9 (2CLK), JK_2_6.9 (2CLK), JK_3_6.9 (2CLK)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: now also SW12_R1.1; no longer SW12_R1.2
- net at ONE_SHOT1.12 (Q_B): now also XOR1.8 (E)
- net at ONE_SHOT1.13 (Q_A): now also XOR1.9 (F)
Other:
- moved on the sheet: 5V_POWER, ONE_SHOT1, SW11_C, SW13_C, SW15_C, SW1_C, SW3_C, SW5_C, SW7_C, SW9_C
